File: Alpaca Fever.sch (KiCad schematic (older format))
At the start: 32 parts, among them J1 INPUT, J2 OUTPUT, J3 SWITCH, J4 +9V, J5 GND, U1 CD4049UBE

Commit message: Cleaned up some connectors and power flags
Connections:
- net +9V: no longer names the net of D100.2 (A), J4.1, LED1.A
Changed lines of the file:
@@
-$EndComp
-$Comp
-L power:+9V #PWR01
-U 1 1 624EA4FC
-P 3300 1050
-F 0 "#PWR01" H 3300 900 50  0001 C CNN
-F 1 "+9V" H 3315 1223 50  0000 C CNN
-F 2 "SparkFun-Connectors:1X01_LONGPAD" H 3300 1050 50  0001 C CNN
-F 3 "" H 3300 1050 50  0001 C CNN
-	1    3300 1050
-	1    0    0    -1
 $EndComp
 $Comp
@@
 $EndComp
 Wire Wire Line
-	3300 1050 3300 1150
-Wire Wire Line
 	4600 1300 4850 1300
 Wire Wire Line
@@
 Wire Wire Line
 	6500 4100 6600 4100
-Wire Wire Line
-	6600 4100 6600 4150
 Wire Wire Line
 	6600 3200 6600 3100
@@
 Wire Wire Line
 	8950 3850 8950 3650
-$Comp
-L power:PWR_FLAG #FLG0101
-U 1 1 62581420
-P 3000 1150
-F 0 "#FLG0101" H 3000 1225 50  0001 C CNN
-F 1 "PWR_FLAG" V 3000 1277 50  0000 L CNN
-F 2 "" H 3000 1150 50  0001 C CNN
-F 3 "~" H 3000 1150 50  0001 C CNN
-	1    3000 1150
-	0    -1   -1   0
-$EndComp
-Connection ~ 3300 1150
 Wire Wire Line
 	3300 1150 3300 1300
-$Comp
-L power:PWR_FLAG #FLG0102
-U 1 1 62586E64
-P 5150 1100
-F 0 "#FLG0102" H 5150 1175 50  0001 C CNN
-F 1 "PWR_FLAG" H 5150 1273 50  0000 C CNN
-F 2 "" H 5150 1100 50  0001 C CNN
-F 3 "~" H 5150 1100 50  0001 C CNN
-	1    5150 1100
-	1    0    0    -1
-$EndComp
-Wire Wire Line
-	5150 1100 4850 1100
-Wire Wire Line
-	4850 1050 4850 1100
-Connection ~ 4850 1100
-Wire Wire Line
-	4850 1100 4850 1300
-$Comp
-L power:PWR_FLAG #FLG0103
-U 1 1 6258B1CF
-P 6650 4150
-F 0 "#FLG0103" H 6650 4225 50  0001 C CNN
-F 1 "PWR_FLAG" H 6650 4323 50  0000 C CNN
-F 2 "" H 6650 4150 50  0001 C CNN
-F 3 "~" H 6650 4150 50  0001 C CNN
-	1    6650 4150
-	1    0    0    -1
-$EndComp
-Wire Wire Line
-	6650 4150 6600 4150
-Connection ~ 6600 4150
-Wire Wire Line
-	6600 4150 6600 4200
 Wire Wire Line
 	3300 1750 3300 1950
@@
 L SparkFun-Connectors:CONN_01 J4
 U 1 1 625974AE
-P 3100 1050
-F 0 "J4" H 3058 1254 45  0001 C CNN
-F 1 "+9V" V 3000 1250 45  0000 R CNN
-F 2 "SparkFun-Connectors:1X01_LONGPAD" H 3100 1250 20  0001 C CNN
-F 3 "" H 3100 1050 50  0001 C CNN
-F 4 "XXX-00000" H 3058 1181 60  0001 C CNN "Field4"
-	1    3100 1050
+P 3300 1050
+F 0 "J4" H 3258 1254 45  0001 C CNN
+F 1 "+9V" V 3200 1250 45  0000 R CNN
+F 2 "SparkFun-Connectors:1X01_LONGPAD" H 3300 1250 20  0001 C CNN
+F 3 "" H 3300 1050 50  0001 C CNN
+F 4 "XXX-00000" H 3258 1181 60  0001 C CNN "Field4"
+	1    3300 1050
 	0    -1   1    0
 $EndComp
@@
 	5200 1950 5550 1950
 Wire Wire Line
-	3000 1150 3100 1150
-Connection ~ 3100 1150
-Wire Wire Line
-	3100 1150 3300 1150
+	6600 4100 6600 4200
+Wire Wire Line
+	4850 1050 4850 1300
 $EndSCHEMATC
